File: hw/power.brd (EAGLE design)
At the start: 61 x 28 mm, 93 parts, among them SW1 MF-SW-TACT-4.2MM, SW2 MF-SW-TACT-4.2MM, U1 TPS54200, U2 TPS54200, U3 TPS54200, U4 TPS54200, U5 MIC280, U6 MIC280, U7 MIC5233, U8 NRF52832, Y1 32MHz, Y2 32.768kHz

Commit message: hw: add few assembly notes and values
Parts:
- R1, R11, R12, R3, R5, R6, R8, R9: value tbd -> 270
Changed lines of the file:
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@@
 <attribute name="VALUE" x="5.6095" y="5.7525" size="0.4064" layer="27" rot="R270"/>
 </element>
-<element name="R1" library="MF_Passives" package="R0805" value="tbd" x="12.2" y="18.6" smashed="yes" rot="R270">
+<element name="R1" library="MF_Passives" package="R0805" value="270" x="12.2" y="18.6" smashed="yes" rot="R270">
 <attribute name="HOUSEPART" value="" x="12.2" y="18.6" size="1.778" layer="27" rot="R270" display="off"/>
 <attribute name="MPN" value="" x="12.2" y="18.6" size="1.778" layer="27" rot="R270" display="off"/>
@@
 <attribute name="WATTAGE" value="" x="12.2" y="18.6" size="1.778" layer="27" rot="R270" display="off"/>
 </element>
-<element name="R3" library="MF_Passives" package="R0805" value="tbd" x="14.2" y="18.6" smashed="yes" rot="R270">
+<element name="R3" library="MF_Passives" package="R0805" value="270" x="14.2" y="18.6" smashed="yes" rot="R270">
 <attribute name="HOUSEPART" value="" x="14.2" y="18.6" size="1.778" layer="27" rot="R270" display="off"/>
 <attribute name="MPN" value="" x="14.2" y="18.6" size="1.778" layer="27" rot="R270" display="off"/>
@@
 <attribute name="VOLTAGE" value="" x="7.4" y="3" size="1.778" layer="27" display="off"/>
 </element>
-<element name="R5" library="MF_Passives" package="R0805" value="tbd" x="29" y="18.6" smashed="yes" rot="R270">
+<element name="R5" library="MF_Passives" package="R0805" value="270" x="29" y="18.6" smashed="yes" rot="R270">
 <attribute name="HOUSEPART" value="" x="4.4" y="43.8" size="1.778" layer="27" rot="R270" display="off"/>
 <attribute name="MPN" value="" x="4.4" y="43.8" size="1.778" layer="27" rot="R270" display="off"/>
@@
 <attribute name="WATTAGE" value="" x="4.4" y="43.8" size="1.778" layer="27" rot="R270" display="off"/>
 </element>
-<element name="R6" library="MF_Passives" package="R0805" value="tbd" x="27" y="18.6" smashed="yes" rot="R270">
+<element name="R6" library="MF_Passives" package="R0805" value="270" x="27" y="18.6" smashed="yes" rot="R270">
 <attribute name="HOUSEPART" value="" x="3" y="29.4" size="1.778" layer="27" rot="R270" display="off"/>
 <attribute name="MPN" value="" x="3" y="29.4" size="1.778" layer="27" rot="R270" display="off"/>
@@
 <attribute name="VOLTAGE" value="" x="17.8" y="3" size="1.778" layer="27" display="off"/>
 </element>
-<element name="R8" library="MF_Passives" package="R0805" value="tbd" x="41.8" y="18.6" smashed="yes" rot="R270">
+<element name="R8" library="MF_Passives" package="R0805" value="270" x="41.8" y="18.6" smashed="yes" rot="R270">
 <attribute name="HOUSEPART" value="" x="21.4" y="29.4" size="1.778" layer="27" rot="R270" display="off"/>
 <attribute name="MPN" value="" x="21.4" y="29.4" size="1.778" layer="27" rot="R270" display="off"/>
@@
 <attribute name="WATTAGE" value="" x="21.4" y="29.4" size="1.778" layer="27" rot="R270" display="off"/>
 </element>
-<element name="R9" library="MF_Passives" package="R0805" value="tbd" x="43.8" y="18.6" smashed="yes" rot="R270">
+<element name="R9" library="MF_Passives" package="R0805" value="270" x="43.8" y="18.6" smashed="yes" rot="R270">
 <attribute name="HOUSEPART" value="" x="19.8" y="33.6" size="1.778" layer="27" rot="R270" display="off"/>
 <attribute name="MPN" value="" x="19.8" y="33.6" size="1.778" layer="27" rot="R270" display="off"/>
@@
 <attribute name="VOLTAGE" value="" x="31.6" y="3" size="1.778" layer="27" display="off"/>
 </element>
-<element name="R11" library="MF_Passives" package="R0805" value="tbd" x="56.6" y="18.6" smashed="yes" rot="R270">
+<element name="R11" library="MF_Passives" package="R0805" value="270" x="56.6" y="18.6" smashed="yes" rot="R270">
 <attribute name="HOUSEPART" value="" x="36.2" y="29.4" size="1.778" layer="27" rot="R270" display="off"/>
 <attribute name="MPN" value="" x="36.2" y="29.4" size="1.778" layer="27" rot="R270" display="off"/>
@@
 <attribute name="WATTAGE" value="" x="36.2" y="29.4" size="1.778" layer="27" rot="R270" display="off"/>
 </element>
-<element name="R12" library="MF_Passives" package="R0805" value="tbd" x="58.6" y="18.6" smashed="yes" rot="R270">
+<element name="R12" library="MF_Passives" package="R0805" value="270" x="58.6" y="18.6" smashed="yes" rot="R270">
 <attribute name="HOUSEPART" value="" x="34.6" y="33.6" size="1.778" layer="27" rot="R270" display="off"/>
 <attribute name="MPN" value="" x="34.6" y="33.6" size="1.778" layer="27" rot="R270" display="off"/>
