File: hw/spotlight.sch (EAGLE design)
At the start: 26 parts, among them J1 LENS-LEDIL-TINA, J2 LENS-LEDIL-TINA, J3 LENS-LEDIL-TINA, J4 LENS-LEDIL-TINA, J5 LENS-LEDIL-TINA, J6 LENS-LEDIL-TINA, U1 MIC280, U2 MIC280

Commit message: hw: add few assembly notes and values
Other:
- note added: "TODO: Change temperature sensors Dual mounting options everywhere Smaller test pads Polarity marking"
- note added: "i2c addr = 0x4a"
- note added: "i2c addr = 0x4b"
