File: hardware/tk-retrofit.brd (EAGLE design)
At the start: 30 x 14 mm, 38 parts, among them U2 DRDC3105, U7 MIC5233, U8 NRF52832, Y1 32MHz, Y2 32.768kHz

Commit message: tk-retrofit: fix ldo p/n
Parts:
- U7: value MIC5233 -> MIC5301
Changed lines of the file:
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@@
 <attribute name="VALUE" x="7.225" y="3.905" size="1.27" layer="27" rot="R270"/>
 </element>
-<element name="U7" library="SparkFun-PowerIC" package="SOT23-5" value="MIC5233" x="4.4" y="9.8" smashed="yes" rot="R270">
+<element name="U7" library="SparkFun-PowerIC" package="SOT23-5" value="MIC5301" x="4.4" y="9.8" smashed="yes" rot="R270">
 <attribute name="NAME" x="6.559" y="10.689" size="0.4064" layer="25" rot="R270"/>
 <attribute name="VALUE" x="4.2095" y="10.7525" size="0.4064" layer="27" rot="R270"/>

Commit message: hw: tk-retrofit: change xtal cap values
Parts:
- C24, C25: value 33p -> 12p
- C26, C27: value 16p -> 12p
Changed lines of the file:
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@@
 <attribute name="VALUE" x="20.768" y="7.124" size="1.27" layer="27" rot="R270"/>
 </element>
-<element name="C24" library="balto" package="0603" value="33p" x="19.6" y="9.8" smashed="yes">
+<element name="C24" library="balto" package="0603" value="12p" x="19.6" y="9.8" smashed="yes">
 <attribute name="NAME" x="18.076" y="10.562" size="1.27" layer="25"/>
 <attribute name="VALUE" x="18.076" y="7.768" size="1.27" layer="27"/>
 </element>
-<element name="C25" library="balto" package="0603" value="33p" x="17.2" y="12.2" smashed="yes" rot="R90">
+<element name="C25" library="balto" package="0603" value="12p" x="17.2" y="12.2" smashed="yes" rot="R90">
 <attribute name="NAME" x="16.438" y="10.676" size="1.27" layer="25" rot="R90"/>
 <attribute name="VALUE" x="19.232" y="10.676" size="1.27" layer="27" rot="R90"/>
 </element>
-<element name="C26" library="balto" package="0603" value="16p" x="9.6" y="12" smashed="yes" rot="R90">
+<element name="C26" library="balto" package="0603" value="12p" x="9.6" y="12" smashed="yes" rot="R90">
 <attribute name="NAME" x="8.838" y="10.476" size="1.27" layer="25" rot="R90"/>
 <attribute name="VALUE" x="11.632" y="10.476" size="1.27" layer="27" rot="R90"/>
 </element>
-<element name="C27" library="balto" package="0603" value="16p" x="7.8" y="6" smashed="yes" rot="R180">
+<element name="C27" library="balto" package="0603" value="12p" x="7.8" y="6" smashed="yes" rot="R180">
 <attribute name="NAME" x="9.324" y="5.238" size="1.27" layer="25" rot="R180"/>
 <attribute name="VALUE" x="9.324" y="8.032" size="1.27" layer="27" rot="R180"/>
