File: hardware/actik-retrofit.brd (EAGLE design)
At the start: 31 x 17 mm, 46 parts, among them U1 TMP102, U5 2450AT18D0100-L, U6 MAX17048, U7 MIC5301, U8 NRF52832, Y4 32.768kHz

Commit message: hw: actik-retrofit: sent to fab, r0
Parts:
- added TP6: TPTP10R, testpad:TP10R
- moved C13 0.20 mm to (15.4, 11.8)
- moved C15 0.20 mm to (20.2, 11.8)
- moved C9 0.20 mm to (16.6, 11.8)
- moved R15 0.20 mm to (17.8, 11.8)
Connections:
- new net IO4: TP6.TP, U8.41
Routing:
- net IO4: track 0.00 -> 2.19 mm
- net +3V3: track 71.8 -> 72.7 mm
- net SDA: track 24.6 -> 25.3 mm
- net SCL: track 26.6 -> 27.3 mm
- net GND: vias 16 -> 53
Other:
- board size 31 x 17 mm -> 31 x 16.4 mm
- board text added: "+"
- board text added: "-"
- board text added: "1"
- board text added: "2"
- board text added: "3"
- board text added: "4"
- board text added: "C"
- board text added: "D"
- board text added: "FB2020"

Commit message: hw: actik-retrofit: add xtal missing value
Parts:
- Y1: value (none) -> 32MHz
Changed lines of the file:
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@@
 <attribute name="VALUE" x="17.8" y="3.7" size="0.6096" layer="27" font="vector" ratio="20" align="top-center"/>
 </element>
-<element name="Y1" library="balto" package="XTAL-2X1.6" value="" x="23.2" y="11.8" smashed="yes" rot="R90">
+<element name="Y1" library="balto" package="XTAL-2X1.6" value="32MHz" x="23.2" y="11.8" smashed="yes" rot="R90">
 <attribute name="NAME" x="22.2" y="9.8" size="1.016" layer="25" rot="R90"/>
 <attribute name="VALUE" x="24.2" y="9.8" size="1.016" layer="27" rot="R90" align="top-left"/>

Commit message: hw: actik: annotate the main decoupling cap
Parts:
- C15: value .1u -> 10u
Changed lines of the file:
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@@
 <attribute name="VALUE" x="14.724" y="4.832" size="1.27" layer="27" rot="R180"/>
 </element>
-<element name="C15" library="balto" package="0603" value=".1u" x="20.2" y="11.8" smashed="yes" rot="R90">
+<element name="C15" library="balto" package="0603" value="10u" x="20.2" y="11.8" smashed="yes" rot="R90">
 <attribute name="NAME" x="19.438" y="0.276" size="1.27" layer="25" rot="R90"/>
 <attribute name="VALUE" x="22.232" y="0.276" size="1.27" layer="27" rot="R90"/>

Commit message: hw: actik: change few R values
Parts:
- R1: value 1k -> 2k2
- R2: value 10k -> 22k
- R3, R6, R7: value 10k -> 12k
Changed lines of the file:
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@@
 <attribute name="VALUE" x="11.4" y="15.5" size="1.27" layer="27" rot="R270"/>
 </element>
-<element name="R1" library="balto" package="0603" value="1k" x="9.8" y="2.4" smashed="yes" rot="R270">
+<element name="R1" library="balto" package="0603" value="2k2" x="9.8" y="2.4" smashed="yes" rot="R270">
 <attribute name="NAME" x="10.562" y="3.924" size="1.27" layer="25" rot="R270"/>
 <attribute name="VALUE" x="7.768" y="3.924" size="1.27" layer="27" rot="R270"/>
@@
 <attribute name="VALUE" x="15.768" y="13.324" size="1.27" layer="27" rot="R270"/>
 </element>
-<element name="R2" library="balto" package="0603" value="10k" x="8.6" y="2.4" smashed="yes" rot="R90">
+<element name="R2" library="balto" package="0603" value="22k" x="8.6" y="2.4" smashed="yes" rot="R90">
 <attribute name="NAME" x="7.838" y="0.876" size="1.27" layer="25" rot="R90"/>
 <attribute name="VALUE" x="10.632" y="0.876" size="1.27" layer="27" rot="R90"/>
@@
 <attribute name="VALUE" x="6.765" y="8.108" size="0.0254" layer="27" rot="R270"/>
 </element>
-<element name="R3" library="balto" package="0603" value="10k" x="22.2" y="4.2" smashed="yes" rot="R90">
+<element name="R3" library="balto" package="0603" value="12k" x="22.2" y="4.2" smashed="yes" rot="R90">
 <attribute name="NAME" x="21.438" y="2.676" size="1.27" layer="25" rot="R90"/>
 <attribute name="VALUE" x="24.232" y="2.676" size="1.27" layer="27" rot="R90"/>
 </element>
-<element name="R6" library="balto" package="0603" value="10k" x="9.8" y="6.8" smashed="yes" rot="R270">
+<element name="R6" library="balto" package="0603" value="12k" x="9.8" y="6.8" smashed="yes" rot="R270">
 <attribute name="NAME" x="10.562" y="8.324" size="1.27" layer="25" rot="R270"/>
 <attribute name="VALUE" x="7.768" y="8.324" size="1.27" layer="27" rot="R270"/>
 </element>
-<element name="R7" library="balto" package="0603" value="10k" x="8.6" y="6.8" smashed="yes" rot="R270">
+<element name="R7" library="balto" package="0603" value="12k" x="8.6" y="6.8" smashed="yes" rot="R270">
 <attribute name="NAME" x="9.362" y="8.324" size="1.27" layer="25" rot="R270"/>
 <attribute name="VALUE" x="6.568" y="8.324" size="1.27" layer="27" rot="R270"/>
