File: hardware/actik-retrofit-r1.brd (EAGLE design)
At the start: 31 x 21.4 mm, 42 parts, among them U13 MAX17055, U5 2450AT18D0100-R, U7 MIC5301, U8 NRF52832, Y1 32MHz, Y4 32.768kHz

Commit message: hw: change few values
Parts:
- C32: value .1u -> 1u
Changed lines of the file:
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@@
 <attribute name="VALUE" x="9.168" y="8.324003125" size="1.27" layer="27" rot="R270"/>
 </element>
-<element name="C32" library="balto" package="0603" value=".1u" x="25" y="8.4" smashed="yes" rot="R180">
+<element name="C32" library="balto" package="0603" value="1u" x="25" y="8.4" smashed="yes" rot="R180">
 <attribute name="NAME" x="26.524" y="7.638" size="1.27" layer="25" rot="R180"/>
 <attribute name="VALUE" x="26.524" y="10.432" size="1.27" layer="27" rot="R180"/>

Commit message: hw: actik-r1 set red led res value
Parts:
- R1: value tbd -> 220
Changed lines of the file:
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@@
 <attribute name="VALUE" x="11.16" y="14.825" size="1.27" layer="27"/>
 </element>
-<element name="R1" library="balto" package="0603" value="tbd" x="11.4" y="10.2" smashed="yes" rot="R180">
+<element name="R1" library="balto" package="0603" value="220" x="11.4" y="10.2" smashed="yes" rot="R180">
 <attribute name="NAME" x="12.924" y="9.438" size="1.27" layer="25" rot="R180"/>
 <attribute name="VALUE" x="12.924" y="12.232" size="1.27" layer="27" rot="R180"/>

Commit message: hw: actik-r1: annotate schematics for antenna tuning values
Parts:
- C8: value dnp -> 1.5p
Changed lines of the file:
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@@
 <?xml version="1.0" encoding="utf-8"?>
 <!DOCTYPE eagle SYSTEM "eagle.dtd">
-<eagle version="9.5.0">
+<eagle version="9.6.2">
 <drawing>
 <settings>
@@
 <attribute name="VALUE" x="21.476" y="4.168" size="1.27" layer="27"/>
 </element>
-<element name="C8" library="balto" package="0603" value="dnp" x="6.6" y="6.8" smashed="yes" rot="R270">
+<element name="C8" library="balto" package="0603" value="1.5p" x="6.6" y="6.8" smashed="yes" rot="R270">
 <attribute name="NAME" x="7.362" y="8.324" size="1.27" layer="25" rot="R270"/>
 <attribute name="VALUE" x="4.568" y="8.324" size="1.27" layer="27" rot="R270"/>
